File: pcb/crobagotchi/crobagotchi.sch (KiCad schematic (older format))
At the start: 10 parts, among them J1 AVR-ISP-6, SW1 SW_Push, SW2 SW_Push, SW3 SW_Push, U1 ATtiny85V-10SU

Commit message: update pcb
Parts:
- added C1: 1uf, Capacitor_SMD:C_1206_3216Metric_Pad1.42x1.75mm_HandSolder, symbol Device:C
- BT1: footprint (none) -> Battery:BatteryHolder_ComfortableElectronic_CH273-2450_1x2450
- Brd1: footprint (none) -> ssd1306:128x64OLED
- J1: footprint (none) -> Connector_PinHeader_2.54mm:PinHeader_2x03_P2.54mm_Vertical
- R1: footprint (none) -> Resistor_SMD:R_1206_3216Metric_Pad1.42x1.75mm_HandSolder
- R2, R3: value 10k -> 4.7K; footprint (none) -> Resistor_SMD:R_1206_3216Metric_Pad1.42x1.75mm_HandSolder
- SW1: footprint (none) -> Jumper:SolderJumper-2_P1.3mm_Open_Pad1.0x1.5mm
- SW2, SW3: footprint (none) -> Button_Switch_THT:SW_PUSH_6mm
Connections:
- net miso is gone; now on net button_option: J1.1 (MISO), U1.6 (PB1)
- net GND: now also SW2.2, SW3.2, C1.2; no longer R2.2, R3.2
- net VCC: now also R2.1, R3.1, C1.1; no longer SW2.2, SW3.2
- net button_option: no longer R2.1, U1.2 (XTAL1/PB3)
- net button_select: now also J1.3 (SCK), U1.7 (PB2); no longer R3.1, U1.3 (XTAL2/PB4)
- net mosi: no longer Brd1.4 (SDA)
- removed net sck: Brd1.3 (SCL), J1.3 (SCK), U1.7 (PB2)
- new net disp_scl: Brd1.3 (SCL), R2.2, U1.2 (XTAL1/PB3)
- new net disp_sda: Brd1.4 (SDA), R3.2, U1.3 (XTAL2/PB4)
Other:
- note removed: "need to update where this conncets, pb0 and pb2 are not the i2c pins"
- moved on the sheet: J1
