File: pcb/crobagotchi/crobagotchi.kicad_pcb (KiCad board)
At the start: 2 copper layers, 33 x 55.9 mm, 11 parts, among them J1 AVR-ISP-6, SW1 SW_Push, SW2 SW_Push, SW3 SW_Push, U1 ATtiny85V-10SU

Commit message: pcb
Parts:
- added svg2mod: G***, crow:kicad_vectorcrob, B.Cu at (108.7, 49.8)
- moved BT1 2.73 mm to (101.1, 68.3)
- moved SW1 1.78 mm to (99.7, 76.2)
- turned R2 to 270 degrees
Routing:
- net VCC: track 0.00 -> 66.7 mm
- net disp_sda: track 0.00 -> 66.5 mm
- net disp_scl: track 0.00 -> 53.3 mm, vias 0 -> 2
- net button_select: track 0.00 -> 45.0 mm, vias 0 -> 2
- net rst: track 0.00 -> 40.6 mm, vias 0 -> 3
- net button_option: track 0.00 -> 39.9 mm, vias 0 -> 2
- net mosi: track 0.00 -> 15.7 mm, vias 0 -> 3
- net GND: track 0.00 -> 4.08 mm, vias 0 -> 2
- added copper zone on B.Cu, net GND
- added copper zone on F.Cu, net GND
Other:
- outline, holes or cut-outs redrawn
- board text added: "A"
- board text added: "B"
- board text added: "Chris Johnston 2021"
- board text added: "Crobagotchi"
- board text added: "Hack me!"
- board text added: "JLCJLCJLCJLC"
- board text added: "Oh no, your screen has been stolen!"
- board text added: "Reset"
